File: hardware/stepper.kicad_pcb (KiCad board)
At the start: 6 copper layers, 40 x 40 mm, 130 parts, among them J101 USB-MINI-B-SMD, J102 DRILL, J103 DRILL, J104 DRILL, J105 DRILL, J401 STACK-UP-HIGH, J402 STACK-DOWN, J403 STACK-UP-HIGH, J404 STACK-DOWN, P201 black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

Commit message: Add heatsink to 3d model
Parts:
- added REF**: heatsink, kicad-libraries:heatsink, F.Cu at (153.2, 93.2)
Changed lines of the file:
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@@
     (links 416)
     (no_connects 2)
-    (area 125.845139 71.945139 283.420502 165.440043)
+    (area 126.671069 72.726549 166.772591 112.825531)
     (thickness 1.6002)
     (drawings 63)
     (tracks 2681)
     (zones 0)
-    (modules 130)
+    (modules 131)
     (nets 149)
   )
@@
     (aux_axis_origin 126.725 72.775)
     (grid_origin 126.725 72.775)
-    (visible_elements FFFFBFFF)
+    (visible_elements FFFF7FFF)
     (pcbplotparams
       (layerselection 0x010fc_8000001f)
@@
     )
   )
-  (module kicad-libraries:TACT-SWITCH (layer Vorderseite)
-    (at 158.2 74.3)
-    (attr smd)
-    (fp_text reference SW101 (at -0.24 -1.79 180) (layer F.Fab)
-      (effects (font (size 0.29972 0.29972) (thickness 0.07493)))
-    )
-    (fp_text value Reset (at -0.04 0 180) (layer F.Fab)
-      (effects (font (size 0.29972 0.29972) (thickness 0.07493)))
-    )
-    (fp_line (start -0.8001 -1.50114) (end -0.8001 -2.10058) (layer F.Fab) (width 0.001))
-    (fp_line (start -0.8001 -2.10058) (end 0.8001 -2.10058) (layer F.Fab) (width 0.001))
-    (fp_line (start 0.8001 -2.10058) (end 0.8001 -1.50114) (layer F.Fab) (width 0.001))
-    (fp_line (start 1.99898 1.50114) (end -1.99898 1.50114) (layer F.Fab) (width 0.001))
-    (fp_line (start -1.99898 1.50114) (end -1.99898 -1.50114) (layer F.Fab) (width 0.001))
-    (fp_line (start -1.99898 -1.50114) (end 1.99898 -1.50114) (layer F.Fab) (width 0.001))
-    (fp_line (start 1.99898 -1.50114) (end 1.99898 1.50114) (layer F.Fab) (width 0.001))
-    (pad 1 smd rect (at -2.09898 0) (size 1.2 1.80086) (layers Vorderseite F.Paste F.Mask)
-      (net 25 STACK-RESET) (clearance 0.14986))
-    (pad 2 smd rect (at 2.09898 0) (size 1.20076 1.80086) (layers Vorderseite F.Paste F.Mask)
-      (net 23 STACK-PGND) (clearance 0.14986))
-    (pad "" thru_hole circle (at 0 0.89916) (size 0.8001 0.8001) (drill 0.8001) (layers *.Cu *.Mask F.SilkS)
-      (clearance 0.14986))
-    (pad "" thru_hole circle (at 0 -0.89916) (size 0.8001 0.8001) (drill 0.8001) (layers *.Cu *.Mask F.SilkS)
-      (clearance 0.14986))
-    (model Buttons_Switches/brick_button_SMD.wrl
-      (at (xyz 0 0 0))
-      (scale (xyz 1 1 1))
-      (rotate (xyz -90 0 0))
-    )
-  )
-  (module kicad-libraries:TACT-SWITCH (layer Vorderseite)
-    (at 135.2 74.3)
-    (attr smd)
-    (fp_text reference SW102 (at -0.24 -1.79 180) (layer F.Fab)
-      (effects (font (size 0.29972 0.29972) (thickness 0.07493)))
-    )
-    (fp_text value Erase (at -0.04 0 180) (layer F.Fab)
-      (effects (font (size 0.29972 0.29972) (thickness 0.07493)))
-    )
-    (fp_line (start -0.8001 -1.50114) (end -0.8001 -2.10058) (layer F.Fab) (width 0.001))
-    (fp_line (start -0.8001 -2.10058) (end 0.8001 -2.10058) (layer F.Fab) (width 0.001))
-    (fp_line (start 0.8001 -2.10058) (end 0.8001 -1.50114) (layer F.Fab) (width 0.001))
-    (fp_line (start 1.99898 1.50114) (end -1.99898 1.50114) (layer F.Fab) (width 0.001))
-    (fp_line (start -1.99898 1.50114) (end -1.99898 -1.50114) (layer F.Fab) (width 0.001))
-    (fp_line (start -1.99898 -1.50114) (end 1.99898 -1.50114) (layer F.Fab) (width 0.001))
-    (fp_line (start 1.99898 -1.50114) (end 1.99898 1.50114) (layer F.Fab) (width 0.001))
-    (pad 1 smd rect (at -2.09898 0) (size 1.2 1.80086) (layers Vorderseite F.Paste F.Mask)
-      (net 108 "Net-(SW102-Pad1)") (clearance 0.14986))
-    (pad 2 smd rect (at 2.09898 0) (size 1.20076 1.80086) (layers Vorderseite F.Paste F.Mask)
-      (net 1 3V3) (clearance 0.14986))
-    (pad "" thru_hole circle (at 0 0.89916) (size 0.8001 0.8001) (drill 0.8001) (layers *.Cu *.Mask F.SilkS)
-      (clearance 0.14986))
-    (pad "" thru_hole circle (at 0 -0.89916) (size 0.8001 0.8001) (drill 0.8001) (layers *.Cu *.Mask F.SilkS)
-      (clearance 0.14986))
-    (model Buttons_Switches/brick_button_SMD.wrl
-      (at (xyz 0 0 0))
-      (scale (xyz 1 1 1))
-      (rotate (xyz -90 0 0))
-    )
-  )
   (module kicad-libraries:LQFP64 (layer Rückseite)
     (at 146.45 82.3)
@@
     )
   )
+  (module kicad-libraries:TACT-SWITCH (layer Vorderseite)
+    (at 135.2 74.3)
+    (attr smd)
+    (fp_text reference SW102 (at -0.24 -1.79 180) (layer F.Fab)
+      (effects (font (size 0.29972 0.29972) (thickness 0.07493)))
+    )
+    (fp_text value Erase (at -0.04 0 180) (layer F.Fab)
+      (effects (font (size 0.29972 0.29972) (thickness 0.07493)))
+    )
+    (fp_line (start -0.8001 -1.50114) (end -0.8001 -2.10058) (layer F.Fab) (width 0.001))
+    (fp_line (start -0.8001 -2.10058) (end 0.8001 -2.10058) (layer F.Fab) (width 0.001))
+    (fp_line (start 0.8001 -2.10058) (end 0.8001 -1.50114) (layer F.Fab) (width 0.001))
+    (fp_line (start 1.99898 1.50114) (end -1.99898 1.50114) (layer F.Fab) (width 0.001))
+    (fp_line (start -1.99898 1.50114) (end -1.99898 -1.50114) (layer F.Fab) (width 0.001))
+    (fp_line (start -1.99898 -1.50114) (end 1.99898 -1.50114) (layer F.Fab) (width 0.001))
+    (fp_line (start 1.99898 -1.50114) (end 1.99898 1.50114) (layer F.Fab) (width 0.001))
+    (pad 1 smd rect (at -2.09898 0) (size 1.2 1.80086) (layers Vorderseite F.Paste F.Mask)
+      (net 108 "Net-(SW102-Pad1)") (clearance 0.14986))
+    (pad 2 smd rect (at 2.09898 0) (size 1.20076 1.80086) (layers Vorderseite F.Paste F.Mask)
+      (net 1 3V3) (clearance 0.14986))
+    (pad "" thru_hole circle (at 0 0.89916) (size 0.8001 0.8001) (drill 0.8001) (layers *.Cu *.Mask F.SilkS)
+      (clearance 0.14986))
+    (pad "" thru_hole circle (at 0 -0.89916) (size 0.8001 0.8001) (drill 0.8001) (layers *.Cu *.Mask F.SilkS)
+      (clearance 0.14986))
+    (model Buttons_Switches/tact_switch_bricks.wrl
+      (at (xyz 0 0 0))
+      (scale (xyz 1 1 1))
+      (rotate (xyz 0 0 180))
+    )
+  )
+  (module kicad-libraries:TACT-SWITCH (layer Vorderseite)
+    (at 158.2 74.3)
+    (attr smd)
+    (fp_text reference SW101 (at -0.24 -1.79 180) (layer F.Fab)
+      (effects (font (size 0.29972 0.29972) (thickness 0.07493)))
+    )
+    (fp_text value Reset (at -0.04 0 180) (layer F.Fab)
+      (effects (font (size 0.29972 0.29972) (thickness 0.07493)))
+    )
+    (fp_line (start -0.8001 -1.50114) (end -0.8001 -2.10058) (layer F.Fab) (width 0.001))
+    (fp_line (start -0.8001 -2.10058) (end 0.8001 -2.10058) (layer F.Fab) (width 0.001))
+    (fp_line (start 0.8001 -2.10058) (end 0.8001 -1.50114) (layer F.Fab) (width 0.001))
+    (fp_line (start 1.99898 1.50114) (end -1.99898 1.50114) (layer F.Fab) (width 0.001))
+    (fp_line (start -1.99898 1.50114) (end -1.99898 -1.50114) (layer F.Fab) (width 0.001))
+    (fp_line (start -1.99898 -1.50114) (end 1.99898 -1.50114) (layer F.Fab) (width 0.001))
+    (fp_line (start 1.99898 -1.50114) (end 1.99898 1.50114) (layer F.Fab) (width 0.001))
+    (pad 1 smd rect (at -2.09898 0) (size 1.2 1.80086) (layers Vorderseite F.Paste F.Mask)
+      (net 25 STACK-RESET) (clearance 0.14986))
+    (pad 2 smd rect (at 2.09898 0) (size 1.20076 1.80086) (layers Vorderseite F.Paste F.Mask)
+      (net 23 STACK-PGND) (clearance 0.14986))
+    (pad "" thru_hole circle (at 0 0.89916) (size 0.8001 0.8001) (drill 0.8001) (layers *.Cu *.Mask F.SilkS)
+      (clearance 0.14986))
+    (pad "" thru_hole circle (at 0 -0.89916) (size 0.8001 0.8001) (drill 0.8001) (layers *.Cu *.Mask F.SilkS)
+      (clearance 0.14986))
+    (model Buttons_Switches/tact_switch_bricks.wrl
+      (at (xyz 0 0 0))
+      (scale (xyz 1 1 1))
+      (rotate (xyz 0 0 180))
+    )
+  )
+  (module kicad-libraries:heatsink (layer Vorderseite)
+    (at 153.175 93.175 90)
+    (fp_text reference REF** (at -0.14 1.79 90) (layer F.Fab)
+      (effects (font (size 1 1) (thickness 0.15)))
+    )
+    (fp_text value heatsink (at 0.13 -2.17 90) (layer F.Fab)
+      (effects (font (size 1 1) (thickness 0.15)))
+    )
+    (fp_line (start -9.74 -6.24) (end 8.59 -6.24) (layer F.Fab) (width 0.15))
+    (fp_line (start 8.59 -6.24) (end 8.58 6.74) (layer F.Fab) (width 0.15))
+    (fp_line (start 8.58 6.74) (end -9.75 6.74) (layer F.Fab) (width 0.15))
+    (fp_line (start -9.75 6.74) (end -9.74 -6.24) (layer F.Fab) (width 0.15))
+    (model unsorted/heatsink.wrl
+      (at (xyz 0 0 0.09))
+      (scale (xyz 1 1 1))
+      (rotate (xyz 0 0 90))
+    )
+  )
